File: docs/eagle/Dew-Point-Control.brd (EAGLE design)
At the start: 100 x 80 mm, 5 parts

Commit message: updated eagle board and schematic
Parts:
- added RELAYS: (no value), pinhead:1X06
Connections:
- new net GPIO17: RELAYS.5, RPI_GPIO.11
- new net GPIO22: RELAYS.3, RPI_GPIO.15
- new net GPIO24: RELAYS.2, RPI_GPIO.18
- new net GPIO27: RELAYS.4, RPI_GPIO.13
- net 5V: now also RELAYS.6
- net GND: now also RELAYS.1
Changed lines of the file:
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@@
 <element name="SENSOR1" library="pinhead" package="1X03" value="" x="24.13" y="69.85" rot="R270"/>
 <element name="SENSOR2" library="pinhead" package="1X03" value="" x="24.13" y="59.69" rot="R270"/>
+<element name="RELAYS" library="pinhead" package="1X06" value="" x="10.16" y="-12.7"/>
 </elements>
 <signals>
@@
 <wire x1="20.32" y1="63.5" x2="24.13" y2="63.5" width="0.4064" layer="16"/>
 <wire x1="24.13" y1="63.5" x2="24.13" y2="62.23" width="0.4064" layer="16"/>
+<contactref element="RELAYS" pad="6"/>
+<wire x1="16.51" y1="-12.7" x2="24.13" y2="62.23" width="0" layer="19" extent="1-1"/>
 </signal>
 <signal name="GND">
@@
 <wire x1="22.86" y1="57.15" x2="12.7" y2="57.15" width="0.4064" layer="16"/>
 <wire x1="12.7" y1="57.15" x2="12.7" y2="66.04" width="0.4064" layer="16"/>
+<contactref element="RELAYS" pad="1"/>
+<wire x1="3.81" y1="-12.7" x2="12.7" y2="57.15" width="0" layer="19" extent="16-16"/>
 </signal>
 <signal name="GPIO18">
@@
 <wire x1="17.78" y1="59.69" x2="24.13" y2="59.69" width="0.4064" layer="16"/>
 </signal>
+<signal name="GPIO24">
+<contactref element="RPI_GPIO" pad="18"/>
+<contactref element="RELAYS" pad="2"/>
+<wire x1="6.35" y1="-12.7" x2="7.62" y2="55.88" width="0" layer="19" extent="1-1"/>
+</signal>
+<signal name="GPIO17">
+<contactref element="RPI_GPIO" pad="11"/>
+<contactref element="RELAYS" pad="5"/>
+<wire x1="13.97" y1="-12.7" x2="5.08" y2="63.5" width="0" layer="19" extent="1-1"/>
+</signal>
+<signal name="GPIO27">
+<contactref element="RPI_GPIO" pad="13"/>
+<contactref element="RELAYS" pad="4"/>
+<wire x1="11.43" y1="-12.7" x2="5.08" y2="60.96" width="0" layer="19" extent="1-1"/>
+</signal>
+<signal name="GPIO22">
+<contactref element="RPI_GPIO" pad="15"/>
+<contactref element="RELAYS" pad="3"/>
+<wire x1="8.89" y1="-12.7" x2="5.08" y2="58.42" width="0" layer="19" extent="1-1"/>
+</signal>
 </signals>

Commit message: rename project and add init script
Connections:
- new net 3,3V: R1.2, R2.2, RPI_GPIO.1, SENSOR1.1, SENSOR2.1
- net 5V: now also RPI_GPIO.2; no longer R1.2, R2.2, RPI_GPIO.1, SENSOR1.1, SENSOR2.1
Routing:
- net 5V: track 55.9 -> 0.00 mm
- net 3,3V: track 0.00 -> 55.9 mm
Changed lines of the file:
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@@
 </elements>
 <signals>
-<signal name="5V">
+<signal name="3,3V">
 <contactref element="RPI_GPIO" pad="1"/>
 <contactref element="SENSOR1" pad="1"/>
@@
 <wire x1="20.32" y1="63.5" x2="24.13" y2="63.5" width="0.4064" layer="16"/>
 <wire x1="24.13" y1="63.5" x2="24.13" y2="62.23" width="0.4064" layer="16"/>
-<contactref element="RELAYS" pad="6"/>
-<wire x1="16.51" y1="-12.7" x2="24.13" y2="62.23" width="0" layer="19" extent="1-1"/>
 </signal>
 <signal name="GND">
@@
 <wire x1="8.89" y1="-12.7" x2="5.08" y2="58.42" width="0" layer="19" extent="1-1"/>
 </signal>
+<signal name="5V">
+<contactref element="RPI_GPIO" pad="2"/>
+<contactref element="RELAYS" pad="6"/>
+<wire x1="16.51" y1="-12.7" x2="7.62" y2="76.2" width="0" layer="19" extent="1-1"/>
+</signal>
 </signals>
